Commit message: Imported upstream version '2.0.1' of 'upstream'

File: turtlebot4_description/urdf/lite/turtlebot4.urdf.xacro (robot description, xacro)
@@ -27,3 +27,11 @@
     <origin xyz="${oakd_lite_x_offset} ${oakd_lite_y_offset} ${oakd_lite_z_offset}"/>
   </xacro:oakd>
+  <!-- Base footprint for navigation -->
+  <link name="base_footprint" />
+  <joint name="base_footprint_joint" type="fixed">
+    <!-- Create3's base_link is already on the ground -->
+    <origin xyz="0 0 0" rpy="0 0 0" />
+    <parent link="base_link" />
+    <child link="base_footprint" />
+  </joint>
 </robot>

File: turtlebot4_description/urdf/sensors/rplidar.urdf.xacro (robot description, xacro)
@@ -30,4 +30,9 @@
   </link>
   <gazebo reference="${name}_link">
+    <!--
+      GPU Ray sensor plugin only supports 180 degrees, so limit to the "front" arc only
+      The lidar is actually mounted sideways on the robot, with +x to the left, so the
+      front arc is actually 0 to -pi
+    -->
     <xacro:ray_sensor sensor_name="${name}" gazebo="${gazebo}"
                   update_rate="62.0" visualize="1"

File: turtlebot4_description/urdf/standard/turtlebot4.urdf.xacro (robot description, xacro)
@@ -101,3 +101,11 @@
     <origin xyz="${oakd_pro_x_offset} ${oakd_pro_y_offset} ${oakd_pro_z_offset}"/>
   </xacro:oakd>
+  <!-- Base footprint for navigation -->
+  <link name="base_footprint" />
+  <joint name="base_footprint_joint" type="fixed">
+    <!-- Create3's base_link is already on the ground -->
+    <origin xyz="0 0 0" rpy="0 0 0" />
+    <parent link="base_link" />
+    <child link="base_footprint" />
+  </joint>
 </robot>
